File: PCB/UI_Board/UI_Board.kicad_sch (KiCad schematic)
At the start: 14 parts, among them J1 DISPLAY, J2 CABLE, SW1 SW_UP, SW2 SW_DWN, SW3 SW_PRE_1, SW4 SW_PRE_2

Commit message: Updated boards
Parts:
- removed R_PU1: 10K, Resistor_THT:R_Axial_DIN0207_L6.3mm_D2.5mm_P7.62mm_Horizontal, symbol Device:R
Connections:
- net 3V3: now also J2.1 (Pin_1); no longer J2.8 (Pin_8)
- net BTNS: now also J2.8 (Pin_8); no longer J2.1 (Pin_1)
- net CS: now also J2.3 (Pin_3); no longer J2.2 (Pin_2)
- net DC: now also J2.7 (Pin_7); no longer J2.3 (Pin_3)
- net GND: now also J2.2 (Pin_2); no longer J2.7 (Pin_7)
- net RST: now also J2.6 (Pin_6); no longer J2.4 (Pin_4)
- net SCL: now also J2.5 (Pin_5); no longer J2.6 (Pin_6)
- net SDA: now also J2.4 (Pin_4); no longer J2.5 (Pin_5)
Changed lines of the file:
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@@
 	)
 	(junction
-		(at 154.94 64.77)
+		(at 162.56 49.53)
 		(diameter 0)
 		(color 0 0 0 0)
 	)
-	(wire
-		(pts
-			(xy 154.94 64.77) (xy 163.83 64.77)
-		)
-		(stroke
-			(width 0)
-			(type default)
-		)
+	(junction
+		(at 153.67 52.07)
+		(diameter 0)
+		(color 0 0 0 0)
 	)
 	(wire
@@
 	(wire
 		(pts
+			(xy 152.4 52.07) (xy 153.67 52.07)
+		)
+		(stroke
+			(width 0)
+			(type default)
+		)
+	)
+	(wire
+		(pts
 			(xy 133.35 104.14) (xy 133.35 107.95)
 		)
@@
 	(wire
 		(pts
-			(xy 158.75 49.53) (xy 163.83 49.53)
+			(xy 162.56 49.53) (xy 163.83 49.53)
 		)
 		(stroke
@@
 	(wire
 		(pts
-			(xy 158.75 54.61) (xy 163.83 54.61)
+			(xy 153.67 52.07) (xy 163.83 52.07)
 		)
 		(stroke
@@
 	(wire
 		(pts
-			(xy 158.75 62.23) (xy 163.83 62.23)
+			(xy 160.02 49.53) (xy 162.56 49.53)
 		)
 		(stroke
@@
 	(wire
 		(pts
-			(xy 143.51 67.31) (xy 163.83 67.31)
-		)
-		(stroke
-			(width 0)
-			(type default)
-		)
-	)
-	(wire
-		(pts
-			(xy 158.75 59.69) (xy 163.83 59.69)
-		)
-		(stroke
-			(width 0)
-			(type default)
-		)
-	)
-	(wire
-		(pts
-			(xy 72.39 67.31) (xy 72.39 71.12)
+			(xy 153.67 52.07) (xy 153.67 53.34)
 		)
 		(stroke
@@
 	(wire
 		(pts
-			(xy 143.51 59.69) (xy 154.94 59.69)
-		)
-		(stroke
-			(width 0)
-			(type default)
-		)
-	)
-	(wire
-		(pts
-			(xy 72.39 78.74) (xy 72.39 83.82)
-		)
-		(stroke
-			(width 0)
-			(type default)
-		)
-	)
-	(wire
-		(pts
 			(xy 114.3 53.34) (xy 116.84 53.34)
 		)
@@
 	(wire
 		(pts
-			(xy 158.75 57.15) (xy 163.83 57.15)
-		)
-		(stroke
-			(width 0)
-			(type default)
-		)
-	)
-	(wire
-		(pts
 			(xy 133.35 91.44) (xy 133.35 96.52)
 		)
@@
 	(wire
 		(pts
-			(xy 158.75 52.07) (xy 163.83 52.07)
-		)
-		(stroke
-			(width 0)
-			(type default)
-		)
-	)
-	(wire
-		(pts
-			(xy 154.94 59.69) (xy 154.94 64.77)
-		)
-		(stroke
-			(width 0)
-			(type default)
-		)
-	)
-	(wire
-		(pts
 			(xy 114.3 91.44) (xy 114.3 107.95)
 		)
@@
 			(width 0)
 			(type default)
-		)
-	)
-	(label "3V3"
-		(at 72.39 67.31 180)
-		(effects
-			(font
-				(size 1.27 1.27)
-			)
-			(justify right bottom)
 		)
 	)
@@
 	)
 	(label "CS"
-		(at 158.75 52.07 180)
+		(at 163.83 54.61 180)
 		(effects
 			(font
@@
 	)
 	(label "DC"
-		(at 158.75 54.61 180)
+		(at 163.83 64.77 180)
 		(effects
 			(font
@@
 	)
 	(label "BTNS"
-		(at 72.39 83.82 180)
-		(effects
-			(font
-				(size 1.27 1.27)
-			)
-			(justify right bottom)
-		)
-	)
-	(label "BTNS"
 		(at 133.35 107.95 180)
 		(effects
@@
 	)
 	(label "SCL"
-		(at 158.75 62.23 180)
+		(at 163.83 59.69 180)
 		(effects
 			(font
@@
 	)
 	(label "3V3"
-		(at 158.75 67.31 180)
+		(at 160.02 49.53 180)
 		(effects
 			(font
@@
 	)
 	(label "SDA"
-		(at 158.75 59.69 180)
+		(at 163.83 57.15 180)
 		(effects
 			(font
@@
 	)
 	(label "RST"
-		(at 158.75 57.15 180)
+		(at 163.83 62.23 180)
 		(effects
 			(font
@@
 	)
 	(label "BTNS"
-		(at 158.75 49.53 180)
+		(at 163.83 67.31 180)
 		(effects
 			(font
@@
 	)
 	(symbol
-		(lib_id "Device:R")
-		(at 72.39 74.93 0)
-		(unit 1)
-		(exclude_from_sim no)
-		(in_bom yes)
-		(on_board yes)
-		(dnp no)
-		(property "Reference" "R_PU1"
-			(at 74.93 73.6599 0)
-			(effects
-				(font
-					(size 1.27 1.27)
-				)
-				(justify left)
-			)
-		)
-		(property "Value" "10K"
-			(at 74.93 76.1999 0)
-			(effects
-				(font
-					(size 1.27 1.27)
-				)
-				(justify left)
-			)
-		)
-		(property "Footprint" "Resistor_THT:R_Axial_DIN0207_L6.3mm_D2.5mm_P7.62mm_Horizontal"
-			(at 70.612 74.93 90)
-			(effects
-				(font
-					(size 1.27 1.27)
-				)
-				(hide yes)
-			)
-		)
-		(property "Datasheet" "~"
-			(at 72.39 74.93 0)
-			(effects
-				(font
-					(size 1.27 1.27)
-				)
-				(hide yes)
-			)
-		)
-		(property "Description" "Resistor"
-			(at 72.39 74.93 0)
-			(effects
-				(font
-					(size 1.27 1.27)
-				)
-				(hide yes)
-			)
-		)
-		(pin "2"
-		)
-		(pin "1"
-		)
-		(instances
-			(project ""
-				(path "/947236bf-2583-4252-8ca1-545b30b49e32"
-					(reference "R_PU1")
-					(unit 1)
-				)
-			)
-		)
-	)
-	(symbol
 		(lib_id "Switch:SW_Push")
 		(at 157.48 91.44 0)
@@
 	(symbol
 		(lib_id "power:GND")
-		(at 154.94 64.77 270)
+		(at 153.67 53.34 0)
 		(unit 1)
 		(exclude_from_sim no)
@@
 		(fields_autoplaced yes)
 		(property "Reference" "#PWR01"
-			(at 148.59 64.77 0)
+			(at 153.67 59.69 0)
 			(effects
 				(font
@@
 		)
 		(property "Value" "GND"
-			(at 151.13 64.7699 90)
-			(effects
-				(font
-					(size 1.27 1.27)
-				)
-				(justify right)
+			(at 153.67 58.42 0)
+			(effects
+				(font
+					(size 1.27 1.27)
+				)
+				(hide yes)
 			)
 		)
 		(property "Footprint" ""
-			(at 154.94 64.77 0)
+			(at 153.67 53.34 0)
 			(effects
 				(font
@@
 		)
 		(property "Datasheet" ""
-			(at 154.94 64.77 0)
+			(at 153.67 53.34 0)
 			(effects
 				(font
@@
 		)
 		(property "Description" "Power symbol creates a global label with name \"GND\" , ground"
-			(at 154.94 64.77 0)
+			(at 153.67 53.34 0)
 			(effects
 				(font
@@
 	(symbol
 		(lib_id "power:PWR_FLAG")
-		(at 143.51 59.69 0)
+		(at 162.56 49.53 0)
 		(unit 1)
 		(exclude_from_sim no)
@@
 		(fields_autoplaced yes)
 		(property "Reference" "#FLG02"
-			(at 143.51 57.785 0)
+			(at 162.56 47.625 0)
 			(effects
 				(font
@@
 		)
 		(property "Value" "PWR_FLAG"
-			(at 143.51 54.61 0)
+			(at 162.56 44.45 0)
 			(effects
 				(font
@@
 		)
 		(property "Footprint" ""
-			(at 143.51 59.69 0)
+			(at 162.56 49.53 0)
 			(effects
 				(font
@@
 		)
 		(property "Datasheet" "~"
-			(at 143.51 59.69 0)
+			(at 162.56 49.53 0)
 			(effects
 				(font
@@
 		)
 		(property "Description" "Special symbol for telling ERC where power comes from"
-			(at 143.51 59.69 0)
+			(at 162.56 49.53 0)
 			(effects
 				(font
@@
 	(symbol
 		(lib_id "power:PWR_FLAG")
-		(at 143.51 67.31 0)
+		(at 152.4 52.07 0)
 		(unit 1)
 		(exclude_from_sim no)
@@
 		(fields_autoplaced yes)
 		(property "Reference" "#FLG01"
-			(at 143.51 65.405 0)
+			(at 152.4 50.165 0)
 			(effects
 				(font
@@
 		)
 		(property "Value" "PWR_FLAG"
-			(at 143.51 62.23 0)
+			(at 152.4 46.99 0)
 			(effects
 				(font
@@
 		)
 		(property "Footprint" ""
-			(at 143.51 67.31 0)
+			(at 152.4 52.07 0)
 			(effects
 				(font
@@
 		)
 		(property "Datasheet" "~"
-			(at 143.51 67.31 0)
+			(at 152.4 52.07 0)
 			(effects
 				(font
@@
 		)
 		(property "Description" "Special symbol for telling ERC where power comes from"
-			(at 143.51 67.31 0)
-			(effects
-				(font
+			(at 152.4 52.07 0)
+			(effects
+				(font
