File: PCB/UI_Board/UI_Board.kicad_sch (KiCad schematic)
At the start: 17 parts, among them J1 DISPLAY, J2 CABLE, SW1 SW_UP, SW2 SW_DWN, SW3 SW_PRE_1, SW4 SW_PRE_2

Commit message: Updated PCB files
Parts:
- removed H1, H2: MountingHole, MountingHole:MountingHole_3.2mm_M3, symbol Mechanical:MountingHole
- added C1: 0.1uF, Capacitor_THT:C_Rect_L7.2mm_W3.5mm_P5.00mm_FKS2_FKP2_MKS2_MKP2, symbol Device:C
Connections:
- net 3V3: now also C1.2
- net GND: now also C1.1
Changed lines of the file:
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@@
 		(color 0 0 0 0)
 	)
-	(wire
-		(pts
-			(xy 118.11 50.8) (xy 118.11 48.26)
-		)
-		(stroke
-			(width 0)
-			(type default)
-		)
+	(junction
+		(at 124.46 45.72)
+		(diameter 0)
+		(color 0 0 0 0)
 	)
 	(wire
@@
 	(wire
 		(pts
+			(xy 133.35 57.15) (xy 123.19 57.15)
+		)
+		(stroke
+			(width 0)
+			(type default)
+		)
+	)
+	(wire
+		(pts
 			(xy 160.02 49.53) (xy 162.56 49.53)
 		)
@@
 	(wire
 		(pts
-			(xy 114.3 50.8) (xy 118.11 50.8)
-		)
-		(stroke
-			(width 0)
-			(type default)
-		)
-	)
-	(wire
-		(pts
 			(xy 153.67 52.07) (xy 153.67 53.34)
 		)
@@
 	(wire
 		(pts
+			(xy 133.35 49.53) (xy 133.35 45.72)
+		)
+		(stroke
+			(width 0)
+			(type default)
+		)
+	)
+	(wire
+		(pts
+			(xy 114.3 45.72) (xy 114.3 50.8)
+		)
+		(stroke
+			(width 0)
+			(type default)
+		)
+	)
+	(wire
+		(pts
 			(xy 181.61 91.44) (xy 181.61 97.79)
 		)
@@
 	(wire
 		(pts
-			(xy 114.3 53.34) (xy 116.84 53.34)
+			(xy 114.3 45.72) (xy 124.46 45.72)
+		)
+		(stroke
+			(width 0)
+			(type default)
+		)
+	)
+	(wire
+		(pts
+			(xy 114.3 53.34) (xy 123.19 53.34)
 		)
 		(stroke
@@
 	(wire
 		(pts
+			(xy 133.35 45.72) (xy 124.46 45.72)
+		)
+		(stroke
+			(width 0)
+			(type default)
+		)
+	)
+	(wire
+		(pts
 			(xy 116.84 60.96) (xy 114.3 60.96)
 		)
@@
 		(pts
 			(xy 133.35 91.44) (xy 133.35 96.52)
+		)
+		(stroke
+			(width 0)
+			(type default)
+		)
+	)
+	(wire
+		(pts
+			(xy 123.19 57.15) (xy 123.19 53.34)
 		)
 		(stroke
@@
 	)
 	(symbol
-		(lib_id "Mechanical:MountingHole")
-		(at 83.82 34.29 0)
+		(lib_id "Device:C")
+		(at 133.35 53.34 0)
 		(unit 1)
 		(exclude_from_sim no)
-		(in_bom no)
+		(in_bom yes)
 		(on_board yes)
 		(dnp no)
 		(fields_autoplaced yes)
-		(property "Reference" "H2"
-			(at 86.36 33.0199 0)
+		(property "Reference" "C1"
+			(at 137.16 52.0699 0)
 			(effects
 				(font
@@
 			)
 		)
-		(property "Value" "MountingHole"
-			(at 86.36 35.5599 0)
+		(property "Value" "0.1uF"
+			(at 137.16 54.6099 0)
 			(effects
 				(font
@@
 			)
 		)
-		(property "Footprint" "MountingHole:MountingHole_3.2mm_M3"
-			(at 83.82 34.29 0)
+		(property "Footprint" "Capacitor_THT:C_Rect_L7.2mm_W3.5mm_P5.00mm_FKS2_FKP2_MKS2_MKP2"
+			(at 134.3152 57.15 0)
 			(effects
 				(font
@@
 		)
 		(property "Datasheet" "~"
-			(at 83.82 34.29 0)
-			(effects
-				(font
-					(size 1.27 1.27)
-				)
-				(hide yes)
-			)
-		)
-		(property "Description" "Mounting Hole without connection"
-			(at 83.82 34.29 0)
-			(effects
-				(font
-					(size 1.27 1.27)
-				)
-				(hide yes)
-			)
+			(at 133.35 53.34 0)
+			(effects
+				(font
+					(size 1.27 1.27)
+				)
+				(hide yes)
+			)
+		)
+		(property "Description" "Unpolarized capacitor"
+			(at 133.35 53.34 0)
+			(effects
+				(font
+					(size 1.27 1.27)
+				)
+				(hide yes)
+			)
+		)
+		(pin "1"
+		)
+		(pin "2"
 		)
 		(instances
-			(project "UI_Board"
+			(project ""
 				(path "/947236bf-2583-4252-8ca1-545b30b49e32"
-					(reference "H2")
+					(reference "C1")
 					(unit 1)
 				)
@@
 	(symbol
 		(lib_id "power:GND")
-		(at 118.11 48.26 180)
+		(at 124.46 45.72 0)
 		(unit 1)
 		(exclude_from_sim no)
@@
 		(fields_autoplaced yes)
 		(property "Reference" "#PWR02"
-			(at 118.11 41.91 0)
+			(at 124.46 52.07 0)
 			(effects
 				(font
@@
 		)
 		(property "Value" "GND"
-			(at 118.11 43.18 0)
+			(at 124.46 50.8 0)
 			(effects
 				(font
@@
 		)
 		(property "Footprint" ""
-			(at 118.11 48.26 0)
+			(at 124.46 45.72 0)
 			(effects
 				(font
@@
 		)
 		(property "Datasheet" ""
-			(at 118.11 48.26 0)
+			(at 124.46 45.72 0)
 			(effects
 				(font
@@
 		)
 		(property "Description" "Power symbol creates a global label with name \"GND\" , ground"
-			(at 118.11 48.26 0)
+			(at 124.46 45.72 0)
 			(effects
 				(font
@@
 					(unit 1)
 				)
-			)
-		)
-	)
-	(symbol
-		(lib_id "Mechanical:MountingHole")
-		(at 73.66 34.29 0)
-		(unit 1)
-		(exclude_from_sim no)
-		(in_bom no)
-		(on_board yes)
-		(dnp no)
-		(fields_autoplaced yes)
-		(property "Reference" "H1"
-			(at 76.2 33.0199 0)
-			(effects
-				(font
-					(size 1.27 1.27)
-				)
-				(justify left)
-			)
-		)
-		(property "Value" "MountingHole"
-			(at 76.2 35.5599 0)
-			(effects
-				(font
-					(size 1.27 1.27)
-				)
-				(justify left)
-			)
-		)
-		(property "Footprint" "MountingHole:MountingHole_3.2mm_M3"
-			(at 73.66 34.29 0)
-			(effects
-				(font
-					(size 1.27 1.27)
-				)
-				(hide yes)
-			)
-		)
-		(property "Datasheet" "~"
-			(at 73.66 34.29 0)
-			(effects
-				(font
-					(size 1.27 1.27)
-				)
-				(hide yes)
-			)
-		)
-		(property "Description" "Mounting Hole without connection"
-			(at 73.66 34.29 0)
-			(effects
-				(font
-					(size 1.27 1.27)
-				)
-				(hide yes)
-			)
-		)
-		(instances
-			(project ""
-				(path "/947236bf-2583-4252-8ca1-545b30b49e32"
-					(reference "H1")
-					(unit 1)
-				)
