File: PCB/Main_Board/Main_Board.kicad_sch (KiCad schematic)
At the start: 33 parts, among them J1 POWER_SUPPLY, J2 LIMIT_SWITCH, J3 ToF, J4 BUCK_IN, J5 BUCK_OUT, J6 ESP32_Left, J7 ESP32_Right, J8 CABLE, J9 MOTOR, U1 74AHCT125

Commit message: Added decoupling capacitor to AHCT
Parts:
- added C7: 0.1uF, Capacitor_THT:C_Rect_L7.2mm_W3.5mm_P5.00mm_FKS2_FKP2_MKS2_MKP2, symbol Device:C
Connections:
- net +5V: now also C7.1
- net GND: now also C7.2
Changed lines of the file:
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@@
 	)
 	(junction
+		(at 218.44 104.14)
+		(diameter 0)
+		(color 0 0 0 0)
+	)
+	(junction
 		(at 27.94 31.75)
 		(diameter 0)
@@
 	(wire
 		(pts
+			(xy 204.47 104.14) (xy 218.44 104.14)
+		)
+		(stroke
+			(width 0)
+			(type default)
+		)
+	)
+	(wire
+		(pts
 			(xy 127 99.06) (xy 129.54 99.06)
 		)
@@
 	(wire
 		(pts
+			(xy 204.47 95.25) (xy 204.47 104.14)
+		)
+		(stroke
+			(width 0)
+			(type default)
+		)
+	)
+	(wire
+		(pts
 			(xy 27.94 25.4) (xy 36.83 25.4)
 		)
@@
 	(wire
 		(pts
+			(xy 204.47 78.74) (xy 204.47 87.63)
+		)
+		(stroke
+			(width 0)
+			(type default)
+		)
+	)
+	(wire
+		(pts
 			(xy 97.79 83.82) (xy 101.6 83.82)
 		)
@@
 	(wire
 		(pts
+			(xy 218.44 78.74) (xy 204.47 78.74)
+		)
+		(stroke
+			(width 0)
+			(type default)
+		)
+	)
+	(wire
+		(pts
 			(xy 40.64 55.88) (xy 40.64 58.42)
 		)
@@
 					(unit 1)
 				)
+			)
+		)
+	)
+	(symbol
+		(lib_id "Device:C")
+		(at 204.47 91.44 0)
+		(mirror y)
+		(unit 1)
+		(exclude_from_sim no)
+		(in_bom yes)
+		(on_board yes)
+		(dnp no)
+		(property "Reference" "C7"
+			(at 210.566 89.408 0)
+			(effects
+				(font
+					(size 1.27 1.27)
+				)
+				(justify left)
+			)
+		)
+		(property "Value" "0.1uF"
+			(at 212.344 91.694 0)
+			(effects
+				(font
+					(size 1.27 1.27)
+				)
+				(justify left)
+			)
+		)
+		(property "Footprint" "Capacitor_THT:C_Rect_L7.2mm_W3.5mm_P5.00mm_FKS2_FKP2_MKS2_MKP2"
+			(at 203.5048 95.25 0)
+			(effects
+				(font
+					(size 1.27 1.27)
+				)
+				(hide yes)
+			)
+		)
+		(property "Datasheet" "~"
+			(at 204.47 91.44 0)
+			(effects
+				(font
+					(size 1.27 1.27)
+				)
+				(hide yes)
+			)
+		)
+		(property "Description" "Unpolarized capacitor"
+			(at 204.47 91.44 0)
+			(effects
+				(font
+					(size 1.27 1.27)
+				)
+				(hide yes)
+			)
+		)
+		(pin "2"
+		)
+		(pin "1"
+		)
+		(instances
+			(project "Main_Board"
+				(path "/ebe5e123-9967-4e9a-99c8-0da7150f1a56"
+					(reference "C7")
+					(unit 1)
+				)
