File: PCB/Main_Board/Main_Board.kicad_pcb (KiCad board)
At the start: 2 copper layers, 100.3 x 115.6 mm, 38 parts, among them J1 POWER_SUPPLY, J2 LIMIT_SWITCH, J3 ToF, J4 BUCK_IN, J5 BUCK_OUT, J6 ESP32_Left, J7 ESP32_Right, J8 CABLE, J9 MOTOR, U1 74AHCT125

Commit message: Updated PCB files
Parts:
- moved H2 3.89 mm to (126.5, 125.0)
- moved H4 3.61 mm to (40.0, 23.5)
- moved H1 3.61 mm to (126.5, 23.5)
- moved H3 3.54 mm to (40.0, 125.0)
Routing:
- net /+5V: track 107.7 -> 111.9 mm, vias 2 -> 1
Other:
- outline, holes or cut-outs redrawn
- board text added: "MoTrotten Main Board v0.0.1 June-26 Carmel Barak"
- board text removed: "MoTrotten Main Board v0.0.1 Feb-26 Carmel Barak"
Changed lines of the file:
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@@
 		(tenting front back)
 		(pcbplotparams
-			(layerselection 0x00000000_00000000_55555555_5755f5ff)
+			(layerselection 0x00000000_00000000_55555555_575555ff)
 			(plot_on_all_layers_selection 0x00000000_00000000_00000000_00000000)
 			(disableapertmacros no)
-			(usegerberextensions no)
+			(usegerberextensions yes)
 			(usegerberattributes yes)
 			(usegerberadvancedattributes yes)
@@
 			(outputformat 1)
 			(mirror no)
-			(drillshape 1)
+			(drillshape 0)
 			(scaleselection 1)
-			(outputdirectory "")
+			(outputdirectory "./")
 		)
 	)
@@
 	(footprint "MountingHole:MountingHole_3.2mm_M3"
 		(layer "F.Cu")
-		(at 129.1 21)
+		(at 126.5 23.5)
 		(descr "Mounting Hole 3.2mm, M3, no annular, generated by kicad-footprint-generator mountinghole.py")
 		(tags "mountinghole M3")
@@
 	(footprint "MountingHole:MountingHole_3.2mm_M3"
 		(layer "F.Cu")
-		(at 129.2 127.8)
+		(at 126.5 125)
 		(descr "Mounting Hole 3.2mm, M3, no annular, generated by kicad-footprint-generator mountinghole.py")
 		(tags "mountinghole M3")
@@
 	(footprint "MountingHole:MountingHole_3.2mm_M3"
 		(layer "F.Cu")
-		(at 37.5 127.5)
+		(at 40 125)
 		(descr "Mounting Hole 3.2mm, M3, no annular, generated by kicad-footprint-generator mountinghole.py")
 		(tags "mountinghole M3")
@@
 	(footprint "MountingHole:MountingHole_3.2mm_M3"
 		(layer "F.Cu")
-		(at 37.3 21.1)
+		(at 40 23.5)
 		(descr "Mounting Hole 3.2mm, M3, no annular, generated by kicad-footprint-generator mountinghole.py")
 		(tags "mountinghole M3")
@@
 		(layer "F.SilkS")
 	)
-	(gr_rect
-		(start 33.02 16.51)
-		(end 133.35 132.08)
+	(gr_arc
+		(start 36.02 132.08)
+		(mid 33.89868 131.20132)
+		(end 33.02 129.08)
+		(stroke
+			(width 0.05)
+			(type default)
+		)
+		(layer "Edge.Cuts")
+	)
+	(gr_line
+		(start 133.35 19.51)
+		(end 133.35 129.08)
 		(stroke
 			(width 0.05)
 			(type default)
 		)
-		(fill no)
 		(layer "Edge.Cuts")
 	)
-	(gr_text "MoTrotten Main Board\nv0.0.1 Feb-26\nCarmel Barak"
+	(gr_arc
+		(start 133.35 129.08)
+		(mid 132.47132 131.20132)
+		(end 130.35 132.08)
+		(stroke
+			(width 0.05)
+			(type default)
+		)
+		(layer "Edge.Cuts")
+	)
+	(gr_line
+		(start 36.02 16.51)
+		(end 130.35 16.51)
+		(stroke
+			(width 0.05)
+			(type default)
+		)
+		(layer "Edge.Cuts")
+	)
+	(gr_line
+		(start 130.35 132.08)
+		(end 36.02 132.08)
+		(stroke
+			(width 0.05)
+			(type default)
+		)
+		(layer "Edge.Cuts")
+	)
+	(gr_arc
+		(start 33.02 19.51)
+		(mid 33.89868 17.38868)
+		(end 36.02 16.51)
+		(stroke
+			(width 0.05)
+			(type default)
+		)
+		(layer "Edge.Cuts")
+	)
+	(gr_line
+		(start 33.02 129.08)
+		(end 33.02 19.51)
+		(stroke
+			(width 0.05)
+			(type default)
+		)
+		(layer "Edge.Cuts")
+	)
+	(gr_arc
+		(start 130.35 16.51)
+		(mid 132.47132 17.38868)
+		(end 133.35 19.51)
+		(stroke
+			(width 0.05)
+			(type default)
+		)
+		(layer "Edge.Cuts")
+	)
+	(gr_text "MoTrotten Main Board\nv0.0.1 June-26\nCarmel Barak"
 		(at 44.45 127 0)
 		(layer "F.SilkS")
@@
 	)
 	(segment
-		(start 82.55 62.23)
-		(end 85.09 62.23)
-		(width 0.25)
+		(start 65.77 59.73)
+		(end 66.5 59)
+		(width 1)
 		(layer "F.Cu")
 		(net 6)
 	)
 	(segment
-		(start 82.5 62.18)
-		(end 82.55 62.23)
-		(width 0.25)
+		(start 82.5 59)
+		(end 82.5 62.18)
+		(width 1)
 		(layer "F.Cu")
 		(net 6)
 	)
 	(segment
-		(start 80.05 59.73)
+		(start 82.5 62.18)
 		(end 82.55 62.23)
-		(width 0.25)
+		(width 1)
 		(layer "F.Cu")
 		(net 6)
 	)
 	(segment
-		(start 64.77 59.73)
-		(end 80.05 59.73)
-		(width 0.25)
+		(start 55.5 88.52)
+		(end 64.77 97.79)
+		(width 1)
 		(layer "F.Cu")
 		(net 6)
 	)
 	(segment
-		(start 85.09 62.23)
-		(end 86.36 63.5)
-		(width 0.25)
+		(start 55.5 51)
+		(end 55.5 88.52)
+		(width 1)
 		(layer "F.Cu")
 		(net 6)
 	)
 	(segment
-		(start 82.5 59)
-		(end 82.5 62.18)
-		(width 0.25)
+		(start 62.5 57.46)
+		(end 64.77 59.73)
+		(width 1)
 		(layer "F.Cu")
 		(net 6)
 	)
 	(segment
-		(start 64.77 58.27)
-		(end 64.77 59.73)
-		(width 0.25)
+		(start 64.77 59.73)
+		(end 65.77 59.73)
+		(width 1)
 		(layer "F.Cu")
 		(net 6)
@@
 	(segment
 		(start 62.5 56)
-		(end 64.77 58.27)
-		(width 0.25)
+		(end 62.5 57.46)
+		(width 1)
 		(layer "F.Cu")
 		(net 6)
 	)
-	(via
-		(at 86.36 63.5)
-		(size 0.6)
-		(drill 0.3)
-		(layers "F.Cu" "B.Cu")
+	(segment
+		(start 66.5 59)
+		(end 82.5 59)
+		(width 1)
+		(layer "F.Cu")
 		(net 6)
 	)
@@
 		(start 64.8 97.6)
 		(end 64.99 97.79)
-		(width 0.25)
+		(width 1)
 		(layer "B.Cu")
 		(net 6)
@@
 		(start 64.77 97.63)
 		(end 64.8 97.6)
-		(width 0.25)
-		(layer "B.Cu")
-		(net 6)
-	)
-	(segment
-		(start 64.99 97.79)
-		(end 90.17 97.79)
-		(width 0.25)
+		(width 1)
 		(layer "B.Cu")
 		(net 6)
 	)
 	(segment
-		(start 93.98 93.98)
-		(end 90.17 97.79)
-		(width 0.25)
+		(start 55.5 51)
+		(end 57.5 51)
+		(width 1)
 		(layer "B.Cu")
 		(net 6)
 	)
 	(segment
-		(start 90.563116 63.5)
-		(end 93.98 66.916884)
-		(width 0.25)
+		(start 57.5 51)
+		(end 62.5 56)
+		(width 1)
 		(layer "B.Cu")
 		(net 6)
@@
 		(start 64.77 97.79)
 		(end 64.77 97.63)
-		(width 0.25)
-		(layer "B.Cu")
-		(net 6)
-	)
-	(segment
-		(start 93.98 66.916884)
-		(end 93.98 93.98)
-		(width 0.25)
+		(width 1)
 		(layer "B.Cu")
 		(net 6)
@@
 		(start 90.17 97.79)
 		(end 90.17 98.17)
-		(width 0.25)
-		(layer "B.Cu")
-		(net 6)
-	)
-	(segment
-		(start 57.5 51)
-		(end 62.5 56)
-		(width 0.25)
+		(width 1)
 		(layer "B.Cu")
 		(net 6)
 	)
 	(segment
-		(start 55.5 51)
-		(end 57.5 51)
-		(width 0.25)
-		(layer "B.Cu")
-		(net 6)
-	)
-	(segment
-		(start 86.36 63.5)
-		(end 90.563116 63.5)
-		(width 0.25)
+		(start 90.17 97.79)
+		(end 64.77 97.79)
+		(width 1)
 		(layer "B.Cu")
 		(net 6)
@@
 		(start 75.09 125.73)
 		(end 75.09 127.49)
-		(width 0.25)
+		(width 0.8)
 		(layer "F.Cu")
 		(net 10)
@@
 		(start 98.53 128.6)
 		(end 101.95 125.18)
-		(width 0.25)
+		(width 0.8)
 		(layer "F.Cu")
 		(net 10)
@@
 		(start 76.2 128.6)
 		(end 98.53 128.6)
-		(width 0.25)
+		(width 0.8)
 		(layer "F.Cu")
 		(net 10)
@@
 		(start 75.09 127.49)
 		(end 76.2 128.6)
-		(width 0.25)
+		(width 0.8)
 		(layer "F.Cu")
 		(net 10)
@@
 		(start 72.31 112.5)
 		(end 75.09 115.28)
-		(width 0.25)
+		(width 0.8)
 		(layer "F.Cu")
 		(net 10)
@@
 		(start 102.82 124.31)
 		(end 101.95 125.18)
-		(width 0.25)
+		(width 0.8)
 		(layer "F.Cu")
 		(net 10)
@@
 		(start 101.95 125.18)
 		(end 101.95 125.05)
-		(width 0.25)
+		(width 0.8)
 		(layer "F.Cu")
 		(net 10)
@@
 		(start 101.95 125.05)
 		(end 102 125)
-		(width 0.25)
+		(width 0.8)
 		(layer "F.Cu")
 		(net 10)
@@
 		(start 75.09 115.28)
 		(end 75.09 125.73)
-		(width 0.25)
+		(width 0.8)
 		(layer "F.Cu")
 		(net 10)
@@
 		(start 102.82 120.6)
 		(end 102.82 124.31)
-		(width 0.25)
+		(width 0.8)
 		(layer "F.Cu")
 		(net 10)
@@
 		(start 90.17 40.33)
 		(end 90.17 49.53)
-		(width 0.25)
+		(width 0.8)
 		(layer "B.Cu")
 		(net 10)
@@
 		(start 93.5 37)
 		(end 100 37)
-		(width 0.25)
+		(width 0.8)
 		(layer "B.Cu")
 		(net 10)
@@
 		(start 93.5 37)
 		(end 90.17 40.33)
-		(width 0.25)
+		(width 0.8)
 		(layer "B.Cu")
 		(net 10)
@@
 		(start 101.95 125.18)
 		(end 101.95 61.31)
-		(width 0.25)
+		(width 0.8)
 		(layer "B.Cu")
 		(net 10)
@@
 		(start 101.95 61.31)
 		(end 90.17 49.53)
-		(width 0.25)
+		(width 0.8)
 		(layer "B.Cu")
 		(net 10)
